Commit message: Merge the two scanners into one 360 degree scan, and measure what it misses
First C++ component, per ADR 0004. The merge geometry is deliberately free of
ROS and TF so it unit tests in milliseconds; the node supplies transforms and
everything else is arithmetic. 14 gtest cases.

Two things the merge does that a naive concatenation of range arrays would not.
Each scan is transformed using the transform that held AT ITS OWN TIMESTAMP,
routed through the odometry frame, because the scanners are not phase locked and
up to 35 ms of vehicle motion at 2 m/s is 70 mm, larger than the 20 mm object
the scanner is specified to detect. And bins take the nearest return, never an
average: averaging a 0.4 m obstacle with a 10 m wall would report 5 m of clear
space that is not there.

Self-returns are dropped by a footprint filter. That is not hypothetical: the
corner scanners see their own chassis at about 0.06 m, measured.

Coverage is measured rather than assumed, and the metric had to be chosen with
care. A count of empty bins is nearly useless, since re-binning polar data from
an off-centre origin at the same angular resolution leaves scattered single-bin
holes that are an artifact. Only a contiguous run is a blind sector.

Measured on the running system, the first attempt left a contiguous 11.56 degree
hole. That turned out to be structural, not a tuning error: from a recessed
position a ray aimed at the opposite corner re-enters the chassis before
clearing it, so seeing tangentially along the vehicle's own side requires the
optics to be at or beyond the envelope corner. The link origin is now the
optical centre, flush at the corner and 5 mm proud, with the housing drawn 60 mm
inboard so the body still sits in the recess and inside the published envelope.
That halved the gap to 4.25 degrees.

It is still short of the sheet's 360 degree claim, and V-06 says so rather than
rounding it away. The residual is vehicle occlusion at grazing incidence and not
a merge error: a unit test drives the same merge with two ideal unoccluded
scanners at the deployed 2118-bin resolution and the largest gap is at most one
bin. The protective field design later must treat those two sectors as
unobserved.

One test had encoded the defect. test_platform_spec asserted the scanner sits
inside the chassis length, which is precisely the arrangement that opens the
blind sector. It now asserts the opposite, and bounds how far proud the optics
may stand before this stops being the platform on the data sheet.

53 tests green, ruff clean, clean build from scratch.

File: src/amr_description/urdf/sensors.xacro (robot description, xacro)
@@ -18,7 +18,20 @@
        result downstream. -->
   <xacro:macro name="safety_scanner" params="name rx ry yaw">
+    <!-- The link origin is the OPTICAL CENTRE, not the centre of the housing.
+         That distinction is the whole reason this mount works.
+         A safety scanner recessed inboard of the vehicle's corner cannot see
+         tangentially along the vehicle's own sides: a ray from an inboard
+         position towards the far corner re-enters the chassis before it clears
+         the body. That is structural, not a tuning error, and it measured as a
+         contiguous 11.6 degree blind sector in the merged scan.
+         Sitting flush at the corner, the optics graze both adjacent faces and
+         see roughly the outward half plane. Two of them on opposite corners
+         then cover the full turn, which is what the platform claims. The
+         housing is drawn inboard so the physical body still sits in the recess
+         and inside the published envelope. -->
     <link name="${name}_link">
       <xacro:box_inertia m="${p['scanner_mass']}" x="${p['scanner_body_x']}" y="${p['scanner_body_y']}" z="${p['scanner_body_z']}"/>
       <visual>
+        <origin xyz="${-p['scanner_housing_inset']} 0 0"/>
         <geometry><box size="${p['scanner_body_x']} ${p['scanner_body_y']} ${p['scanner_body_z']}"/></geometry>
         <material name="amr_sensor"/>
