Commit message: Validation pass: fix a malformed TF tree, a misplaced centre of mass, and a test that lied
An audit of everything built so far, checking claims against the running system
rather than against my own notes. Six real defects, each now covered by a gate
that was verified to fail when the defect is reintroduced.

The TF tree was malformed. The description carried base_footprint as a child of
base_link while diff_drive_controller published odom -> base_footprint, so that
frame had two parents, one static and one dynamic. Nothing warned. base_link
already sits on the ground plane at the centre of the drive axis, so
base_footprint was an exact duplicate of it and is simply gone;
base_frame_id is now the root link. A test asserts that invariant directly.

The chassis centre of mass sat at ground level. box_inertia emitted no origin,
so the mass of the body was placed at the link origin while its geometry is
centred 163 mm higher. That lowers the centre of mass by the full body half
height and makes the robot markedly harder to tip than the real machine, which
would have quietly flattered every payload and cornering result later. A test
now requires the inertial origin to coincide with the geometry.

drive_check was not repeatable. Run twice in a row, the second run started its
acceleration ramp at roughly 1.75 m/s left over from the first and reported
reaching top speed in 4.99 m at an effective 0.35 m/s2, above the limit the
controller enforces. It read like a physics finding and was measurement error:
the check commanded zero for a fixed number of spins instead of waiting for the
robot to stop. It now blocks on an actual rest condition, and two back-to-back
runs are identical.

CI would have failed on its first run: eight ruff findings in code I had
written and never linted locally.

The README carried a stale provenance count, claiming 20 datasheet values, 4
derived and 10 estimated when the spec had grown to 54 constants at 29, 5 and
20. A project whose whole claim is that numbers are traceable cannot carry a
wrong count of them. Same for the test count.

Benchmark precision was overstated. Re-running after the inertia change, the
cheap configurations move by about 8 percent between runs because their per-step
cost is a small difference between two larger wall times. Those rows are now
quoted to two significant digits; the expensive rows that the tier split
actually turns on repeat to within a few percent.

Also records what the model does NOT do, in docs/validation.md: caster joint
states are not published so their frames are absent from TF, scan_time is zero
on the laser messages, there is no jerk limit, the camera field of view is the
optimistic reading of an ambiguous sheet, and the CMake dev warning on build
comes from upstream and is left alone rather than papered over with a local
policy that does not reach the scope raising it.

File: src/amr_description/urdf/amr.urdf.xacro (robot description, xacro)
@@ -71,5 +71,6 @@
                        x="${p['chassis_length']}"
                        y="${p['chassis_width']}"
-                       z="${body_h}"/>
+                       z="${body_h}"
+                       cz="${body_cz}"/>
     <visual>
       <origin xyz="0 0 ${body_cz}"/>
@@ -86,12 +87,13 @@
     </collision>
   </link>
-  <!-- Ground projection frame. Nav2 and the costmaps work in this frame; the
-       inertial body is base_link above it. -->
-  <link name="base_footprint"/>
-  <joint name="base_footprint_joint" type="fixed">
-    <parent link="base_link"/>
-    <child link="base_footprint"/>
-    <origin xyz="0 0 0"/>
-  </joint>
+  <!-- There is deliberately NO base_footprint link.
+       base_link already sits on the ground plane at the centre of the drive
+       axis, so a base_footprint would be an exact duplicate of it. Worse, it
+       was actively broken: the description made it a CHILD of base_link while
+       diff_drive_controller published odom -> base_footprint, giving that frame
+       two parents and a malformed TF tree. Nothing warned. Nav2's default
+       robot_base_frame is base_link, so this costs nothing.
+       test_description.py asserts the controller's base_frame_id is the root
+       link, which is the invariant that was violated. -->
   <!-- Load deck: the surface a top module or a KLT sits on. Named so the
        payload work in a later phase has a frame to attach to. -->

File: src/amr_description/urdf/inertia.xacro (robot description, xacro)
@@ -8,7 +8,14 @@
      construction. -->
 <robot xmlns:xacro="http://www.ros.org/wiki/xacro">
-  <!-- Solid cuboid about its centre of mass. -->
-  <xacro:macro name="box_inertia" params="m x y z">
+  <!-- Solid cuboid. `cz` places the centre of mass along the link Z axis; it
+       MUST match wherever the visual and collision geometry actually sit.
+       Leaving it at the link origin puts the mass somewhere the body is not:
+       the chassis centre of mass ended up 163 mm below the body, at ground
+       level between the wheels, which makes the robot far harder to tip than
+       the real machine and would have flattered every payload and cornering
+       result. -->
+  <xacro:macro name="box_inertia" params="m x y z cz:=0">
     <inertial>
+      <origin xyz="0 0 ${cz}"/>
       <mass value="${m}"/>
       <inertia
@@ -22,4 +29,5 @@
   <xacro:macro name="wheel_inertia" params="m r width">
     <inertial>
+      <origin xyz="0 0 0"/>
       <mass value="${m}"/>
       <inertia

Commit message: Make the vehicle occlude its own scanners
The scanners sat inside a chassis modelled as one solid 800 x 580 box, with the
nearest wall 40 mm away in x and 30 mm in y, both below the 50 mm minimum range.
The scans looked entirely healthy: 1618 returns, no infinities, 0.27 m minimum,
5 m median. Nothing suggested a problem.

The renderer culls backfaces, so a sensor inside a box sees no box, and the
vehicle was invisible to its own lidar. Probing the arc aimed into the robot
made it plain: 159 returns with a median of 9.34 m, which is the scanner looking
straight through the chassis at the far wall of the warehouse.

Every later claim about 360 degree coverage, protective field geometry or blind
sectors would have rested on that artifact.

The chassis is now two overlapping boxes forming a plus shape, leaving the four
corners open as recesses for the scanners. Both boxes stay inside the published
800 x 580 mm envelope, the sensors sit in open corners rather than buried in
solid geometry, and the remaining body is a real occluder. Measured after the
change, the same inward arc returns a median of 0.06 m, the chassis wall, while
the outward arc is unchanged at 4.57 m.

Inertia is still taken over the full envelope rather than the plus shape. The
recesses are a small fraction of the volume and the bounding box slightly
over-estimates the yaw moment, which is the conservative direction for turning.
Stated in the description rather than left implicit.

This also turns the self-footprint filter in the scan merge from an anticipated
requirement into a demonstrated one: those 0.06 m returns are real and have to
be removed before the merged scan is usable.

File: src/amr_description/urdf/amr.urdf.xacro (robot description, xacro)
@@ -68,4 +68,8 @@
        the geometric centre of the footprint. -->
   <link name="base_link">
+    <!-- Inertia is taken over the full 800 x 580 envelope rather than the plus
+         shape. The corner recesses are a small fraction of the volume and the
+         bounding box slightly over-estimates the yaw moment, which is the
+         conservative direction for turning. Approximation, stated. -->
     <xacro:box_inertia m="${body_mass}"
                        x="${p['chassis_length']}"
@@ -73,16 +77,32 @@
                        z="${body_h}"
                        cz="${body_cz}"/>
-    <visual>
-      <origin xyz="0 0 ${body_cz}"/>
-      <geometry>
-        <box size="${p['chassis_length']} ${p['chassis_width']} ${body_h}"/>
-      </geometry>
+    <!-- The chassis is TWO overlapping boxes, not one, forming a plus shape that
+         leaves the four corners open. Those recesses house the safety scanners.
+         This is not styling. With a single solid box the scanners sit inside it,
+         and because the renderer culls backfaces a sensor inside a box makes
+         that box invisible: measured on the running system, rays aimed into the
+         vehicle returned a median of 9.34 m, seeing straight through the robot
+         to the far wall. The vehicle has to be a real occluder or every claim
+         about scanner coverage rests on a rendering artifact.
+         Both boxes stay inside the published 800 x 580 mm envelope. -->
+    <xacro:property name="body_long_w" value="${p['chassis_width'] - 2 * p['corner_cut_y']}"/>
+    <xacro:property name="body_wide_l" value="${p['chassis_length'] - 2 * p['corner_cut_x']}"/>
+    <visual name="body_longitudinal">
+      <origin xyz="0 0 ${body_cz}"/>
+      <geometry><box size="${p['chassis_length']} ${body_long_w} ${body_h}"/></geometry>
       <material name="amr_body"/>
     </visual>
-    <collision>
-      <origin xyz="0 0 ${body_cz}"/>
-      <geometry>
-        <box size="${p['chassis_length']} ${p['chassis_width']} ${body_h}"/>
-      </geometry>
+    <visual name="body_transverse">
+      <origin xyz="0 0 ${body_cz}"/>
+      <geometry><box size="${body_wide_l} ${p['chassis_width']} ${body_h}"/></geometry>
+      <material name="amr_body"/>
+    </visual>
+    <collision name="body_longitudinal">
+      <origin xyz="0 0 ${body_cz}"/>
+      <geometry><box size="${p['chassis_length']} ${body_long_w} ${body_h}"/></geometry>
+    </collision>
+    <collision name="body_transverse">
+      <origin xyz="0 0 ${body_cz}"/>
+      <geometry><box size="${body_wide_l} ${p['chassis_width']} ${body_h}"/></geometry>
     </collision>
   </link>

Commit message: Fix the things that were visibly wrong, and record what is still broken
Four real defects, found by looking at the running system rather than at the
tests, which were all passing throughout.

The GUIs would not open at all. A terminal from the VS Code snap exports
GTK_PATH into /snap/code, GTK loads snap modules, and those pull in the core20
libpthread; every windowed binary dies with undefined symbol __libc_pthread_init.
The launch now clears that one variable.

The robot rendered as a featureless slab. Its wheels were entirely inside the
chassis box, so nothing showed how it moved, and the casters never rendered at
all because their joint states were not published, which is also why RViz
reported RobotModel Status: Error. The chassis now has real wheel wells, the
wheels carry a rim so their rotation is visible, the casters publish state
interfaces (state only, never commanded, since they are passive), and there is a
signal beacon.

Cameras were switched off in the demo launch, so the sensor suite the whole
perception phase depends on was not present.

Pedestrians tipped over, climbed the racking and then hovered. The cause was
inertia: they carried a real person's centre of mass at 0.95 m over a 0.22 m
collision puck, which tips at about 13 degrees of lean. The inertia now matches
the body that actually touches the floor. They also gained arms and a hi-vis
band, having been a torso on sticks.

STILL BROKEN, and stated rather than hidden: the walkers only travel 0.12 to
0.14 m of their lanes instead of walking them end to end, and one spawns on top
of warehouse clutter. Animated pedestrians are not working. See the plan.

Two process failures worth recording. Killing the people launch does NOT remove
the models it spawned from Gazebo, so every respawn after the first was a no-op
against an existing name and several rounds of measurements were taken against
stale models that never carried the fix under test. And declaring a <gui> block
in the world to aim the camera replaces Gazebo's entire default layout, leaving
every panel floating over the viewport; the camera is now aimed through the
move_to service instead, which leaves the layout alone.

125 tests green, but the tests never had anything to say about any of this.

File: src/amr_description/urdf/amr.urdf.xacro (robot description, xacro)
@@ -57,5 +57,5 @@
   <xacro:property name="component_mass"
     value="${2*p['drive_wheel_mass'] + 4*(p['caster_wheel_mass'] + p['caster_swivel_mass'])
-             + scanner_total + camera_total + p['imu_mass']}"/>
+             + scanner_total + camera_total + p['imu_mass'] + p['beacon_mass']}"/>
   <xacro:property name="body_mass" value="${total_mass - component_mass}"/>
   <material name="amr_body">    <color rgba="0.16 0.17 0.19 1.0"/></material>
@@ -63,4 +63,7 @@
   <material name="amr_dark">    <color rgba="0.05 0.05 0.06 1.0"/></material>
   <material name="amr_sensor">  <color rgba="0.30 0.31 0.33 1.0"/></material>
+  <material name="amr_beacon">  <color rgba="0.95 0.75 0.10 1.0"/></material>
+  <material name="amr_tyre">    <color rgba="0.08 0.08 0.09 1.0"/></material>
+  <material name="amr_rim">     <color rgba="0.55 0.57 0.60 1.0"/></material>
   <!-- ================= chassis ================= -->
   <!-- base_link sits at the centre of the drive wheel axis, projected to the
@@ -88,4 +91,12 @@
     <xacro:property name="body_long_w" value="${p['chassis_width'] - 2 * p['corner_cut_y']}"/>
     <xacro:property name="body_wide_l" value="${p['chassis_length'] - 2 * p['corner_cut_x']}"/>
+    <!-- Wheel wells. The drive wheels sit at the middle of each side, and
+         without a cutout the chassis box simply swallows them: the robot
+         renders as a featureless slab with no visible means of moving. The
+         transverse section is therefore split into a front and a rear block,
+         leaving the middle of each flank open. -->
+    <xacro:property name="well_half" value="${p['drive_wheel_width'] + 0.055}"/>
+    <xacro:property name="block_len" value="${body_wide_l / 2.0 - well_half}"/>
+    <xacro:property name="block_off" value="${well_half + block_len / 2.0}"/>
     <visual name="body_longitudinal">
       <origin xyz="0 0 ${body_cz}"/>
@@ -93,8 +104,22 @@
       <material name="amr_body"/>
     </visual>
-    <visual name="body_transverse">
-      <origin xyz="0 0 ${body_cz}"/>
-      <geometry><box size="${body_wide_l} ${p['chassis_width']} ${body_h}"/></geometry>
+    <visual name="body_front">
+      <origin xyz="${block_off} 0 ${body_cz}"/>
+      <geometry><box size="${block_len} ${p['chassis_width']} ${body_h}"/></geometry>
       <material name="amr_body"/>
+    </visual>
+    <visual name="body_rear">
+      <origin xyz="${-block_off} 0 ${body_cz}"/>
+      <geometry><box size="${block_len} ${p['chassis_width']} ${body_h}"/></geometry>
+      <material name="amr_body"/>
+    </visual>
+    <!-- An accent band around the waist, which is what makes a low slab read as
+         a vehicle rather than a crate. -->
+    <visual name="body_band">
+      <origin xyz="0 0 ${p['ground_clearance'] + body_h * 0.72}"/>
+      <geometry>
+        <box size="${p['chassis_length'] + 0.004} ${body_long_w + 0.004} 0.022"/>
+      </geometry>
+      <material name="amr_accent"/>
     </visual>
     <collision name="body_longitudinal">
@@ -102,9 +127,28 @@
       <geometry><box size="${p['chassis_length']} ${body_long_w} ${body_h}"/></geometry>
     </collision>
-    <collision name="body_transverse">
-      <origin xyz="0 0 ${body_cz}"/>
-      <geometry><box size="${body_wide_l} ${p['chassis_width']} ${body_h}"/></geometry>
+    <collision name="body_front">
+      <origin xyz="${block_off} 0 ${body_cz}"/>
+      <geometry><box size="${block_len} ${p['chassis_width']} ${body_h}"/></geometry>
+    </collision>
+    <collision name="body_rear">
+      <origin xyz="${-block_off} 0 ${body_cz}"/>
+      <geometry><box size="${block_len} ${p['chassis_width']} ${body_h}"/></geometry>
     </collision>
   </link>
+  <!-- Signal beacon. ISO 3691-4 wants the vehicle state visible from outside,
+       and it also gives the silhouette something above the deck line. -->
+  <link name="beacon_link">
+    <xacro:box_inertia m="${p['beacon_mass']}" x="0.06" y="0.06" z="0.09" cz="0.045"/>
+    <visual>
+      <origin xyz="0 0 0.045"/>
+      <geometry><cylinder radius="0.035" length="0.09"/></geometry>
+      <material name="amr_beacon"/>
+    </visual>
+  </link>
+  <joint name="beacon_joint" type="fixed">
+    <parent link="base_link"/>
+    <child link="beacon_link"/>
+    <origin xyz="${-p['chassis_length'] / 2.0 + 0.09} 0 ${p['chassis_height'] + 0.005}"/>
+  </joint>
   <!-- There is deliberately NO base_footprint link.
        base_link already sits on the ground plane at the centre of the drive
@@ -137,10 +181,20 @@
                            r="${p['drive_wheel_radius']}"
                            width="${p['drive_wheel_width']}"/>
-      <visual>
+      <visual name="tyre">
         <origin rpy="${pi/2} 0 0"/>
         <geometry>
           <cylinder radius="${p['drive_wheel_radius']}" length="${p['drive_wheel_width']}"/>
         </geometry>
-        <material name="amr_dark"/>
+        <material name="amr_tyre"/>
+      </visual>
+      <!-- A rim proud of the tyre, so the wheel reads as a wheel and its
+           rotation is visible when the robot drives. -->
+      <visual name="rim">
+        <origin rpy="${pi/2} 0 0"/>
+        <geometry>
+          <cylinder radius="${p['drive_wheel_radius'] * 0.55}"
+                    length="${p['drive_wheel_width'] + 0.006}"/>
+        </geometry>
+        <material name="amr_rim"/>
       </visual>
       <collision>

File: src/amr_description/urdf/ros2_control.xacro (robot description, xacro)
@@ -6,6 +6,12 @@
      hardware. The predecessor used libgazebo_ros_diff_drive, which is both
      Gazebo Classic only and impossible to carry to hardware.
-     The casters are deliberately NOT in ros2_control. They are passive; the
-     physics engine turns them. Declaring them would imply they are actuated. -->
+     The casters carry STATE interfaces only, never a command interface. That
+     distinction is the whole point: they are passive, the physics engine turns
+     them, and nothing commands them. But their angles do have to be published,
+     because otherwise robot_state_publisher cannot place those links, RViz
+     reports RobotModel Status: Error, and the casters do not render at all,
+     which made the vehicle look like a slab with no wheels.
+     On real hardware a caster has no encoder, so this is simulator-only
+     telemetry and is recorded as such in docs/validation.md. -->
 <robot xmlns:xacro="http://www.ros.org/wiki/xacro">
   <xacro:macro name="amr_ros2_control" params="sim ns">
@@ -40,4 +46,18 @@
         <state_interface name="velocity"/>
       </joint>
+      <xacro:macro name="passive_joint" params="name">
+        <joint name="${name}">
+          <state_interface name="position"/>
+          <state_interface name="velocity"/>
+        </joint>
+      </xacro:macro>
+      <xacro:passive_joint name="caster_front_left_swivel_joint"/>
+      <xacro:passive_joint name="caster_front_left_wheel_joint"/>
+      <xacro:passive_joint name="caster_front_right_swivel_joint"/>
+      <xacro:passive_joint name="caster_front_right_wheel_joint"/>
+      <xacro:passive_joint name="caster_rear_left_swivel_joint"/>
+      <xacro:passive_joint name="caster_rear_left_wheel_joint"/>
+      <xacro:passive_joint name="caster_rear_right_swivel_joint"/>
+      <xacro:passive_joint name="caster_rear_right_wheel_joint"/>
     </ros2_control>
     <xacro:if value="${sim}">

Commit message: SLAM works: it was an unmanaged lifecycle node all along
Three separate faults, and not one of them logged an error. The node ran, the
scan was healthy at 3102 returns a frame, and nothing appeared on /map.

The merged scan was malformed: angle_max equalled angle_min plus 2*pi, so the
first and last ray described the same bearing and a consumer stepping by
angle_increment gets one ray too many. Fixed with a test. Not the cause.

The scan had no frame of its own. Its frame_id was base_link, which is also
slam_toolbox's base_frame, leaving the laser transform as identity. The merged
scan is now published in base_scan. Also not the cause.

async_slam_toolbox_node is a LIFECYCLE node and nothing was managing it. It sat
in unconfigured indefinitely, which is why it declared no parameters at all:
ros2 param get returned Parameter not set and the node logged only Failed to get
parameters: resolution. A lifecycle manager now brings it up. That was the
cause.

The diagnostic that cracked it was ros2 lifecycle get, which is the same check
that cracked the identical problem on nav2_collision_monitor earlier. A silent
node should be checked for lifecycle state before anything else, and that is now
written into the validation record.

Result: a 276 x 414 grid at 5 cm, 88.1 m2 mapped free and 1.9 m2 occupied, with
map to odom published. RViz keeps odom as its fixed frame on purpose so the view
still works when slam is disabled, while the Map display renders regardless.

File: src/amr_description/urdf/amr.urdf.xacro (robot description, xacro)
@@ -160,4 +160,17 @@
        test_description.py asserts the controller's base_frame_id is the root
        link, which is the invariant that was violated. -->
+  <!-- Frame the MERGED scan is published in.
+       Coincident with base_link by construction, because the merge already
+       resolves both scanners into base_link coordinates. It exists as a
+       separate frame because a laser whose frame_id IS the SLAM base frame
+       leaves slam_toolbox computing an identity laser transform, and it then
+       accepts the scan and publishes no map at all, silently. A sensor should
+       have its own frame regardless. -->
+  <link name="base_scan"/>
+  <joint name="base_scan_joint" type="fixed">
+    <parent link="base_link"/>
+    <child link="base_scan"/>
+    <origin xyz="0 0 ${p['scanner_mount_height']}"/>
+  </joint>
   <!-- Load deck: the surface a top module or a KLT sits on. Named so the
        payload work in a later phase has a frame to attach to. -->
