Commit message: Model the carried load and measure what it does to braking
Two of the four ISO 13855 terms are braking, and the deceleration comes
from a single 2.4 m/s2 rating the MP-400 manual does not distinguish by
load, unlike the MiR250 sheet whose 0.3 m/s2 is explicitly a
with-maximum-payload figure. The fields have therefore been sized
identically empty and laden on an inherited assumption.

                        unladen 88 kg    laden 188 kg
  samples                        385             474
  p50                           9 mm            9 mm
  p95                          25 mm           19 mm
  fastest stop      85 mm from 0.77   97 mm from 0.89 m/s
  implied decel            3.49 m/s2       4.08 m/s2

Adding 100 kg changed the median by nothing. The treatment was verified on
the live parameter server, 188.00 kg total with a 100 kg payload link,
because V-49's control arm taught that habit.

The reason is architectural rather than a simulator artefact. A protective
stop does not pass through the velocity smoother: the collision monitor
sits downstream of it and zeroes the command outright, so max_decel of
-1.00 m/s2, whose own comment reads "capped below the emergency rate",
never applies to the stop it was written for. The vehicle stops as hard as
the drive and floor allow, which at these speeds is not mass limited.

Measured deceleration exceeds the 2.4 m/s2 the fields assume, so the
v^2/2a term is conservative by a third. NOTHING IS RESIZED ON THIS. A
conservative term is a safe term and V-42 and V-45 are what shrinking a
field costs when the argument is arithmetic. The value is that the term is
checked and the direction of the error is known.

The load is modelled as mass, not as a transfer. DetachableJoint starts
attached and gz-sim 8.11 has no suppress_initial_attach, so a joint cannot
be made where a box was set down and re-made when the vehicle returns.
Pretending otherwise would have been a mechanism, not a measurement.

top_plate_height joins the specs with provenance. The MP-400 manual
publishes H2 at 381 mm and it was quoted inside another key's provenance
while being used nowhere; the load rests on it rather than on the 411 mm
H1, and the 30 mm matters because centre of mass height is the part that
changes behaviour under braking.

File: src/amr_description/urdf/amr.urdf.xacro (robot description, xacro)
@@ -31,4 +31,13 @@
   <xacro:arg name="use_scanners" default="true"/>
   <xacro:arg name="use_cameras"  default="true"/>
+  <!-- PAYLOAD ON THE TOP PLATE, in kilograms, 0 for an empty vehicle.
+       WHY THIS IS A MASS AND NOT A PICK AND PLACE. Gazebo's DetachableJoint
+       starts attached and gz-sim 8.11 has no suppress_initial_attach, so a
+       joint cannot be created where a box was set down and re-made when the
+       vehicle returns for the next one. Modelling the carried mass directly
+       measures the thing that matters, which is what 100 kg does to the
+       braking distance a protective field is sized from, without pretending
+       to a transfer mechanism that is not simulated. See V-60. -->
+  <xacro:arg name="payload_kg"   default="0.0"/>
   <!-- Namespace, normalised to either "" or "name/" so it can be prefixed to a
        topic without callers having to remember the slash. -->
@@ -59,4 +68,9 @@
              + scanner_total + camera_total + p['imu_mass'] + p['beacon_mass']}"/>
   <xacro:property name="body_mass" value="${total_mass - component_mass}"/>
+  <!-- The payload is its OWN link with its own inertia rather than being added
+       to body_mass, because where the load sits changes the yaw moment and the
+       height of the centre of mass, and adding it to the chassis box would
+       silently place 100 kg at the chassis centroid instead of on the deck. -->
+  <xacro:property name="payload_mass" value="${float('$(arg payload_kg)')}"/>
   <material name="amr_body">    <color rgba="0.16 0.17 0.19 1.0"/></material>
   <material name="amr_accent">  <color rgba="0.90 0.55 0.10 1.0"/></material>
@@ -310,3 +324,42 @@
   <!-- ================= actuation and simulation ================= -->
   <xacro:amr_ros2_control sim="$(arg sim)" ns="${ns}"/>
+  <!-- ================= payload ================= -->
+  <!-- A CARRIED LOAD, ON THE PLATE, WITH ITS OWN INERTIA.
+       Built only when payload_kg is above zero, so an empty vehicle is exactly
+       the vehicle it was before this existed and every figure measured without
+       a load stays comparable.
+       The load is modelled as a 400 x 400 mm box on the top plate. That is a
+       Euro half pallet footprint, which is what a 100 kg load on a vehicle
+       this size actually is, and it is centred on the drive axis so the mass
+       does not shift the yaw moment asymmetrically. A real load would not be
+       centred; measuring an off centre one is a separate experiment and this
+       one deliberately isolates mass from balance.
+       Height is taken so the box SITS on the plate rather than being centred
+       on it, because a 100 kg mass 200 mm too low would understate the centre
+       of mass rise, which is the part that matters for tipping and for how the
+       vehicle behaves under braking. -->
+  <xacro:if value="${payload_mass > 0.0}">
+    <xacro:property name="pl_side" value="0.400"/>
+    <xacro:property name="pl_h"    value="0.200"/>
+    <link name="payload">
+      <xacro:box_inertia m="${payload_mass}" x="${pl_side}" y="${pl_side}"
+                         z="${pl_h}" cz="${pl_h / 2.0}"/>
+      <visual>
+        <origin xyz="0 0 ${pl_h / 2.0}"/>
+        <geometry><box size="${pl_side} ${pl_side} ${pl_h}"/></geometry>
+        <material name="amr_accent"/>
+      </visual>
+      <!-- NO COLLISION GEOMETRY, and that is deliberate rather than an
+           oversight. The scanners sit at 110 mm and the plate is at 381 mm, so
+           the load is above every scan plane and cannot be seen by the vehicle
+           itself. Giving it collision would let it catch on racking the
+           protective fields were never sized to clear, which would measure the
+           model rather than the vehicle. The mass and inertia are the point. -->
+    </link>
+    <joint name="payload_joint" type="fixed">
+      <parent link="base_link"/>
+      <child link="payload"/>
+      <origin xyz="0 0 ${p['top_plate_height']}"/>
+    </joint>
+  </xacro:if>
 </robot>
